File: hardware/power_control/power_control/power_control.kicad_pcb (KiCad board)
At the start: 2 copper layers, 20.3 x 28.6 mm, 23 parts, among them J1 Conn_01x03, J2 Conn_01x03, J3 Conn_01x04, J4 Conn_01x06, J5 Conn_01x02, J6 Conn_01x06, SW1 SW_Push, U1 MCP1703A-5002_SOT23, U2 ATtiny1604-SS

Commit message: cosmetic changes: net names and component values
Connections:
- net Net-(C2-Pad1) renamed /VBAT_DIV
- net Net-(J3-Pad3) renamed /UPDI_TX
- net Net-(J5-Pad1) renamed /PBTN
- net Net-(J6-Pad2) renamed /PSYS_CTRL
- net Net-(J6-Pad5) renamed /PMTR_CTRL
- net Net-(R5-Pad1) renamed /PWR_BUTTON
