File: hardware/power_control/power_control/power_control.sch (KiCad schematic (older format))
At the start: 23 parts, among them J1 Conn_01x03, J2 Conn_01x03, J3 Conn_01x04, J4 Conn_01x06, J5 Conn_01x02, J6 Conn_01x06, SW1 SW_Push, U1 MCP1703A-5002_SOT23, U2 ATtiny1604-SS

Commit message: cosmetic changes: net names and component values
Parts:
- C1, C3, C4: value C -> 2.2u
- C2, C5: value C -> 100n
- R1: value R_Small_US -> 330k
- R10, R11, R7, R8, R9: value R_Small_US -> 10k
- R2: value R_Small_US -> 1M
- R3: value R_Small_US -> 4.7k
- R5: value R_Small_US -> 1k
Connections:
- net PSYS_CTRL: now reaches J6.2 (Pin_2), R9.1, U2.11 (PA1)
- net PMTR_CTRL: now reaches J6.5 (Pin_5), R7.1, U2.12 (PA2)
- net VBAT_DIV: now reaches C2.1, R1.1, R2.2, U2.2 (PA4)
- net PWR_BUTTON: now reaches R5.1, U2.5 (PA7)
- net PBTN: now reaches J5.1 (Pin_1), R5.2, R8.1, SW1.1
- net UPDI_TX: now reaches J3.3 (Pin_3), R3.1
Changed lines of the file:
@@
 U 1 1 612492EC
 P 5850 3500
-F 0 "U2" H 5850 4381 50  0000 C CNN
-F 1 "ATtiny1604-SS" H 5850 4290 50  0000 C CNN
+F 0 "U2" H 5450 4150 50  0000 C CNN
+F 1 "ATtiny1604-SS" H 6150 4200 50  0000 C CNN
 F 2 "Package_SO:SOIC-14_3.9x8.7mm_P1.27mm" H 5850 3500 50  0001 C CIN
 F 3 "http://ww1.microchip.com/downloads/en/DeviceDoc/ATtiny804_1604-Data-Sheet-40002028A.pdf" H 5850 3500 50  0001 C CNN
@@
 P 3650 2900
 F 0 "C1" H 3765 2946 50  0000 L CNN
-F 1 "C" H 3765 2855 50  0000 L CNN
+F 1 "2.2u" H 3765 2855 50  0000 L CNN
 F 2 "Capacitor_SMD:C_0603_1608Metric_Pad1.08x0.95mm_HandSolder" H 3688 2750 50  0001 C CNN
 F 3 "~" H 3650 2900 50  0001 C CNN
@@
 P 4650 2900
 F 0 "C3" H 4765 2946 50  0000 L CNN
-F 1 "C" H 4765 2855 50  0000 L CNN
+F 1 "2.2u" H 4765 2855 50  0000 L CNN
 F 2 "Capacitor_SMD:C_0603_1608Metric_Pad1.08x0.95mm_HandSolder" H 4688 2750 50  0001 C CNN
 F 3 "~" H 4650 2900 50  0001 C CNN
@@
 P 4000 4400
 F 0 "C2" H 4115 4446 50  0000 L CNN
-F 1 "C" H 4115 4355 50  0000 L CNN
+F 1 "100n" H 4115 4355 50  0000 L CNN
 F 2 "Capacitor_SMD:C_0603_1608Metric_Pad1.08x0.95mm_HandSolder" H 4038 4250 50  0001 C CNN
 F 3 "~" H 4000 4400 50  0001 C CNN
@@
 U 1 1 612524CE
 P 3750 4350
-F 0 "R1" H 3818 4396 50  0000 L CNN
-F 1 "R_Small_US" H 3818 4305 50  0000 L CNN
+F 0 "R1" H 3600 4400 50  0000 L CNN
+F 1 "330k" H 3500 4300 50  0000 L CNN
 F 2 "Resistor_SMD:R_0603_1608Metric_Pad0.98x0.95mm_HandSolder" H 3750 4350 50  0001 C CNN
 F 3 "~" H 3750 4350 50  0001 C CNN
@@
 P 3900 3900
 F 0 "R2" H 3968 3946 50  0000 L CNN
-F 1 "R_Small_US" H 3968 3855 50  0000 L CNN
+F 1 "1M" H 3968 3855 50  0000 L CNN
 F 2 "Resistor_SMD:R_0603_1608Metric_Pad0.98x0.95mm_HandSolder" H 3900 3900 50  0001 C CNN
 F 3 "~" H 3900 3900 50  0001 C CNN
@@
 P 7800 4000
 F 0 "R8" H 7732 3954 50  0000 R CNN
-F 1 "R_Small_US" H 7732 4045 50  0000 R CNN
+F 1 "10k" H 7732 4045 50  0000 R CNN
 F 2 "Resistor_SMD:R_0603_1608Metric_Pad0.98x0.95mm_HandSolder" H 7800 4000 50  0001 C CNN
 F 3 "~" H 7800 4000 50  0001 C CNN
@@
 P 7850 1850
 F 0 "R9" H 7918 1896 50  0000 L CNN
-F 1 "R_Small_US" H 7918 1805 50  0000 L CNN
+F 1 "10k" H 7918 1805 50  0000 L CNN
 F 2 "Resistor_SMD:R_0603_1608Metric_Pad0.98x0.95mm_HandSolder" H 7850 1850 50  0001 C CNN
 F 3 "~" H 7850 1850 50  0001 C CNN
@@
 P 9000 1200
 F 0 "R11" H 9068 1246 50  0000 L CNN
-F 1 "R_Small_US" H 9068 1155 50  0000 L CNN
+F 1 "10k" H 9068 1155 50  0000 L CNN
 F 2 "Resistor_SMD:R_0603_1608Metric_Pad0.98x0.95mm_HandSolder" H 9000 1200 50  0001 C CNN
 F 3 "~" H 9000 1200 50  0001 C CNN
@@
 P 8650 1200
 F 0 "R10" H 8718 1246 50  0000 L CNN
-F 1 "R_Small_US" H 8718 1155 50  0000 L CNN
+F 1 "10k" H 8718 1155 50  0000 L CNN
 F 2 "Resistor_SMD:R_0603_1608Metric_Pad0.98x0.95mm_HandSolder" H 8650 1200 50  0001 C CNN
 F 3 "~" H 8650 1200 50  0001 C CNN
@@
 P 7650 2500
 F 0 "R7" H 7718 2546 50  0000 L CNN
-F 1 "R_Small_US" H 7718 2455 50  0000 L CNN
+F 1 "10k" H 7718 2455 50  0000 L CNN
 F 2 "Resistor_SMD:R_0603_1608Metric_Pad0.98x0.95mm_HandSolder" H 7650 2500 50  0001 C CNN
 F 3 "~" H 7650 2500 50  0001 C CNN
@@
 U 1 1 61283593
 P 6400 5850
-F 0 "R3" V 6195 5850 50  0000 C CNN
-F 1 "R_Small_US" V 6286 5850 50  0000 C CNN
+F 0 "R3" V 6450 5700 50  0000 C CNN
+F 1 "4.7k" V 6500 5850 50  0000 C CNN
 F 2 "Resistor_SMD:R_0603_1608Metric_Pad0.98x0.95mm_HandSolder" H 6400 5850 50  0001 C CNN
 F 3 "~" H 6400 5850 50  0001 C CNN
@@
 P 7500 4150
 F 0 "R5" V 7705 4150 50  0000 C CNN
-F 1 "R_Small_US" V 7614 4150 50  0000 C CNN
+F 1 "1k" V 7614 4150 50  0000 C CNN
 F 2 "Resistor_SMD:R_0603_1608Metric_Pad0.98x0.95mm_HandSolder" H 7500 4150 50  0001 C CNN
 F 3 "~" H 7500 4150 50  0001 C CNN
@@
 P 5150 1700
 F 0 "C4" H 5265 1746 50  0000 L CNN
-F 1 "C" H 5265 1655 50  0000 L CNN
+F 1 "2.2u" H 5265 1655 50  0000 L CNN
 F 2 "Capacitor_SMD:C_0603_1608Metric_Pad1.08x0.95mm_HandSolder" H 5188 1550 50  0001 C CNN
 F 3 "~" H 5150 1700 50  0001 C CNN
@@
 P 5500 1700
 F 0 "C5" H 5615 1746 50  0000 L CNN
-F 1 "C" H 5615 1655 50  0000 L CNN
+F 1 "100n" H 5615 1655 50  0000 L CNN
 F 2 "Capacitor_SMD:C_0603_1608Metric_Pad1.08x0.95mm_HandSolder" H 5538 1550 50  0001 C CNN
 F 3 "~" H 5500 1700 50  0001 C CNN
@@
 NoConn ~ 6450 3600
 NoConn ~ 6450 3700
+Text Label 7500 1650 0    50   ~ 0
+PSYS_CTRL
+Text Label 7550 2350 0    50   ~ 0
+PMTR_CTRL
+Text Label 4550 4150 0    50   ~ 0
+VBAT_DIV
+Text Label 6900 3800 0    50   ~ 0
+PWR_BUTTON
+Text Label 8350 4150 0    50   ~ 0
+PBTN
+Text Label 6550 5850 0    50   ~ 0
+UPDI_TX
 $EndSCHEMATC
